File: Door.kicad_pcb (KiCad board)
At the start: 2 copper layers, 20.3 x 57.1 mm, 27 parts, among them J101 Programming, J102 Battery input, Q101 NDS355AN, Q201 BSS83P, Q202 BC817, SW101 FLASH, SW102 RESET, SW103 SW_Reed, U101 ESP-12F, U301 TPL5111

Commit message: Revision 1.2
Parts:
- Q101: value NDS355AN -> IRLML6402
- U301: value TPL5111 -> TPL5110
- moved REF** 2.99 mm to (139.1, 66.7)
- turned R107 to 270 degrees
Connections:
- C101 pad 1: +3V3 -> VLOAD
- C301 pad 2: GBAT -> GND
- J102 pad 1: GBAT -> GND
- Q101 pad 1: /timer/DRV_OUT -> Net-(Q101-Pad1)
- Q101 pad 2: GBAT -> +3V3
- Q101 pad 3: GND -> VLOAD
- Q202 pad 2: GBAT -> GND
- R101 pad 1: +3V3 -> VLOAD
- R102 pad 1: +3V3 -> VLOAD
- R103 pad 1: +3V3 -> VLOAD
- R104 pad 1: +3V3 -> VLOAD
- R107 pad 1: GND -> Net-(Q101-Pad1)
- R107 pad 2: /MSW -> /timer/DRV_OUT
- R202 pad 2: GBAT -> GND
- R301 pad 2: GBAT -> GND
- U101 pad 10: Net-(U101-Pad10) -> (no net)
- U101 pad 11: Net-(U101-Pad11) -> (no net)
- U101 pad 12: Net-(U101-Pad12) -> (no net)
- U101 pad 13: Net-(U101-Pad13) -> (no net)
- U101 pad 14: Net-(U101-Pad14) -> (no net)
- U101 pad 19: Net-(U101-Pad19) -> /GP_TIMER
- U101 pad 20: Net-(U101-Pad20) -> /EN_BAT
- U101 pad 5: /EN_BAT -> (no net)
- U101 pad 6: /GP_TIMER -> (no net)
- U101 pad 8: +3V3 -> VLOAD
- U101 pad 9: Net-(U101-Pad9) -> (no net)
- U301 pad 2: GBAT -> GND
- U301 pad 6: GBAT -> GND
Routing:
- net GND: track 68.7 -> 132.2 mm, vias 3 -> 2
- net GBAT: track 41.8 -> 0.00 mm
- net VLOAD: track 0.00 -> 37.0 mm, vias 0 -> 2
- net +3V3: track 72.7 -> 45.8 mm
- net /timer/DRV_OUT: track 0.54 -> 18.2 mm, vias 0 -> 2
- net Net-(Q101-Pad1): track 0.00 -> 13.3 mm, vias 0 -> 2
- net /EN_BAT: track 23.8 -> 32.3 mm, vias 0 -> 2
- net /TX: track 60.3 -> 52.5 mm
- net /RST: track 36.1 -> 42.5 mm
- net /RX: track 53.6 -> 47.6 mm
- net /GP_TIMER: track 35.3 -> 30.6 mm
- net /EN: track 17.6 -> 21.2 mm
- net /GP0: track 37.3 -> 34.8 mm
- net Net-(Q201-Pad1): track 20.5 -> 22.0 mm, vias 2 -> 3
- net /GP2: track 10.9 -> 12.2 mm
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Other:
- rule solder_mask_min_width: 0.15 -> 0.1
- board text added: "REV 1.1"
- board text removed: "REV 1.0"
