File: Door.sch (KiCad schematic (older format))
At the start: 16 parts, among them J101 Programming, J102 Battery input, Q101 NDS355AN, SW101 FLASH, SW102 RESET, SW103 SW_Reed, U101 ESP-12F

Commit message: Revision 1.2
Parts:
- removed Q101: NDS355AN, Package_TO_SOT_SMD:SOT-23, symbol custom:NDS355AN
- removed R107: 10K, Resistor_SMD:R_0805_2012Metric, symbol Device:R
Connections:
- net GBAT is gone; now on net GND: J102.1 (Pin_1)
- net +3V3: no longer C101.1, R101.1, R102.1, R103.1, R104.1, U101.8 (VCC)
- net EN_BAT: now also U101.20 (GPIO5); no longer U101.5 (GPIO14)
- net GND: now also R108.2; no longer R108.1
- net GP_TIMER: now also R108.1, U101.19 (GPIO4); no longer R108.2, U101.6 (GPIO12)
- net GP15: no longer names the net of R106.2, U101.16 (GPIO15)
- new net VLOAD: C101.1, R101.1, R102.1, R103.1, R104.1, U101.8 (VCC)
Other:
- note removed: "Pull downs\n"
- moved on the sheet: R105, R106, R108, SW101, SW102, SW103
