File: battery.sch (KiCad schematic (older format))
At the start: 6 parts, among them Q201 BSS83P, Q202 BC817

Commit message: Revision 1.2
Connections:
- net GBAT renamed GND
Changed lines of the file:
@@
 EESchema Schematic File Version 4
 LIBS:Door-cache
-EELAYER 26 0
+EELAYER 29 0
 EELAYER END
 $Descr A4 11693 8268
 encoding utf-8
 Sheet 2 3
-Title "Vermicompost board"
-Date "2019-02-02"
-Rev ""
+Title "Battery status monitor"
+Date "2019-04-27"
+Rev "1.2"
 Comp "Viktor Stískala"
 Comment1 ""
@@
 	1    0    0    -1
 $EndComp
-Text GLabel 6650 4550 2    50   Input ~ 0
-GBAT
+$Comp
+L power:GND #PWR0202
+U 1 1 5CC5A0B2
+P 6650 4550
+F 0 "#PWR0202" H 6650 4300 50  0001 C CNN
+F 1 "GND" H 6655 4377 50  0000 C CNN
+F 2 "" H 6650 4550 50  0001 C CNN
+F 3 "" H 6650 4550 50  0001 C CNN
+	1    6650 4550
+	-1   0    0    1
+$EndComp
 $EndSCHEMATC
